Commit message: add laser sensor on UR3, but due to collision the sensor was always shaking. Need to be fixed.

File: src/drivers/universal_robot/ur_description/urdf/ur3.urdf.xacro (robot description, xacro)
@@ -356,4 +356,5 @@
       <parent link="${prefix}ee_link" />
       <child link="${prefix}vacuum_gripper" />
+      <child link="hokuyo_joint" />
       <origin rpy="0 1.5708 0" xyz="0.059 0.0535 0" />
       <limit effort="50" velocity="50" lower="0" upper="0" />
@@ -369,4 +370,66 @@
         <minDistance>0.01</minDistance>
       </plugin>
+    </gazebo>
+    <joint name="hokuyo_joint" type="fixed">
+      <axis xyz="0 1 0" />
+      <origin xyz="0 0 0" rpy="0 0 0"/>
+      <parent link="${prefix}vacuum_gripper"/>
+      <child link="hokuyo_link"/>
+    </joint>
+    <!-- Hokuyo Laser -->
+    <link name="hokuyo_link">
+      <collision>
+        <origin xyz="0 0 0" rpy="0 0 0"/>
+        <geometry>
+      <box size="0.1 0.1 0.1"/>
+        </geometry>
+      </collision>
+      <visual>
+        <origin xyz="0 0 0" rpy="0 0 0"/>
+        <geometry>
+          <mesh filename="package://ur_description/meshes/ur3/visual/hokuyo.dae"/>
+        </geometry>
+      </visual>
+      <inertial>
+        <mass value="1e-5" />
+        <origin xyz="0 0 0" rpy="0 0 0"/>
+        <inertia ixx="1e-6" ixy="0" ixz="0" iyy="1e-6" iyz="0" izz="1e-6" />
+      </inertial>
+    </link>
+      <!-- hokuyo -->
+    <gazebo reference="hokuyo_link">
+      <sensor type="gpu_ray" name="head_hokuyo_sensor">
+        <pose>0 0 0 0 0 0</pose>
+        <visualize>false</visualize>
+        <update_rate>40</update_rate>
+        <ray>
+          <scan>
+            <horizontal>
+              <samples>720</samples>
+              <resolution>1</resolution>
+              <min_angle>-1.570796</min_angle>
+              <max_angle>1.570796</max_angle>
+            </horizontal>
+          </scan>
+          <range>
+            <min>0.10</min>
+            <max>30.0</max>
+            <resolution>0.01</resolution>
+          </range>
+          <noise>
+            <type>gaussian</type>
+            <!-- Noise parameters based on published spec for Hokuyo laser
+                achieving "+-30mm" accuracy at range < 10m.  A mean of 0.0m and
+                stddev of 0.01m will put 99.7% of samples within 0.03m of the true
+                reading. -->
+            <mean>0.0</mean>
+            <stddev>0.01</stddev>
+          </noise>
+        </ray>
+        <plugin name="gazebo_ros_head_hokuyo_controller" filename="libgazebo_ros_gpu_laser.so">
+          <topicName>/rrbot/laser/scan</topicName>
+          <frameName>hokuyo_link</frameName>
+        </plugin>
+      </sensor>
     </gazebo>
     <xacro:ur_arm_transmission prefix="${prefix}" hw_interface="${transmission_hw_interface}" />

Commit message: Add files via upload

File: src/drivers/universal_robot/ur_description/urdf/ur3.urdf.xacro (robot description, xacro)
@@ -373,6 +373,6 @@
     <joint name="hokuyo_joint" type="fixed">
       <axis xyz="0 1 0" />
-      <origin xyz="0 0 0" rpy="0 0 0"/>
-      <parent link="${prefix}vacuum_gripper"/>
+      <origin xyz="0.1 0 0" rpy="0 1.570796 0"/>
+      <parent link="${prefix}ee_link"/>
       <child link="hokuyo_link"/>
     </joint>
@@ -399,7 +399,7 @@
       <!-- hokuyo -->
     <gazebo reference="hokuyo_link">
-      <sensor type="gpu_ray" name="head_hokuyo_sensor">
+      <sensor type="ray" name="head_hokuyo_sensor">
         <pose>0 0 0 0 0 0</pose>
-        <visualize>false</visualize>
+        <visualize>true</visualize>
         <update_rate>40</update_rate>
         <ray>
@@ -427,5 +427,5 @@
           </noise>
         </ray>
-        <plugin name="gazebo_ros_head_hokuyo_controller" filename="libgazebo_ros_gpu_laser.so">
+        <plugin name="gazebo_ros_head_hokuyo_controller" filename="libgazebo_ros_laser.so">
           <topicName>/rrbot/laser/scan</topicName>
           <frameName>hokuyo_link</frameName>

Commit message: Update Documentation to Sphinx format. Update ur3.urdf.xacro, optimize the sensor location and collision model.

File: src/drivers/universal_robot/ur_description/urdf/ur3.urdf.xacro (robot description, xacro)
@@ -373,5 +373,5 @@
     <joint name="hokuyo_joint" type="fixed">
       <axis xyz="0 1 0" />
-      <origin xyz="0.1 0 0" rpy="0 1.570796 0"/>
+      <origin xyz="0.00 -0.015 0" rpy="0.0 1.570796 0.0"/>
       <parent link="${prefix}ee_link"/>
       <child link="hokuyo_link"/>
@@ -379,10 +379,10 @@
     <!-- Hokuyo Laser -->
     <link name="hokuyo_link">
-      <collision>
+      <!-- <collision>
         <origin xyz="0 0 0" rpy="0 0 0"/>
         <geometry>
       <box size="0.1 0.1 0.1"/>
         </geometry>
-      </collision>
+      </collision> -->
       <visual>
         <origin xyz="0 0 0" rpy="0 0 0"/>
